File: splinky-shield.kicad_pcb (KiCad board)
At the start: 2 copper layers, 73.5 x 50.8 mm, 57 parts, among them J1 USB_C_Receptacle_USB2.0, J10 Ribbon, J11 Serial, J12 Conn_01x04_Female, J2 Conn_01x04_Female, J3 Conn_01x04_Female, J4 Conn_01x04_Female, J5 Conn_01x02, J6 Serial, J7 trackball, J8 Ribbon, J9 RGB, SW1 SW_SPST, SW3 SW_SPST, U1 RP2040, U2 GD25Q80CEIGR, U3 XC6210B332MR-G, U4 USBLC6-2P6, Y1 Crystal_GND24

Commit message: drc
Parts:
- moved FB1 0.97 mm to (187.5, 92.9)
Routing:
- net Net-(FB1-Pad2): track 24.7 -> 25.7 mm
Changed lines of the file:
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@@
   )
   (footprint "Inductor_SMD:L_0603_1608Metric" (layer "F.Cu")
-    (at 187.41 91.92 90)
+    (at 187.53 92.88 90)
     (descr "Inductor SMD 0603 (1608 Metric), square (rectangular) end terminal, IPC_7351 nominal, (Body size source: http://www.tortai-tech.com/upload/download/2011102023233369053.pdf), generated with kicad-footprint-generator")
     (tags "inductor")
@@
   (segment (start 155.55 90.5) (end 155.55 85.79) (width 0.16) (layer "F.Cu") (net 10))
   (via (at 155.55 90.5) (size 0.6) (drill 0.3) (layers "F.Cu" "B.Cu") (net 10))
-  (segment (start 186.585 88.496) (end 186.585 90.3075) (width 0.4) (layer "F.Cu") (net 11))
-  (segment (start 186.585 90.3075) (end 187.41 91.1325) (width 0.4) (layer "F.Cu") (net 11))
+  (segment (start 186.585 88.496) (end 186.585 91.1475) (width 0.4) (layer "F.Cu") (net 11))
+  (segment (start 186.585 91.1475) (end 187.53 92.0925) (width 0.4) (layer "F.Cu") (net 11))
   (segment (start 196.061 90.17) (end 197.735 88.496) (width 0.4) (layer "B.Cu") (net 11))
   (segment (start 188.259 90.17) (end 196.061 90.17) (width 0.4) (layer "B.Cu") (net 11))
@@
   (segment (start 146.85 90.35) (end 147.55 90.35) (width 0.16) (layer "F.Cu") (net 53))
   (segment (start 192.7075 93.847991) (end 192.7075 94.459513) (width 0.2) (layer "F.Cu") (net 63))
+  (segment (start 185.575 94.95) (end 192.217013 94.95) (width 0.2) (layer "F.Cu") (net 63))
   (segment (start 191.185489 90.926073) (end 191.41 90.701562) (width 0.2) (layer "F.Cu") (net 63))
   (segment (start 192.729511 91.089511) (end 192.729511 92.12598) (width 0.2) (layer "F.Cu") (net 63))
   (segment (start 191.003929 92.526824) (end 191.185489 92.345264) (width 0.2) (layer "F.Cu") (net 63))
   (segment (start 192.547013 94.62) (end 193.257013 93.91) (width 0.2) (layer "F.Cu") (net 63))
-  (segment (start 187.85 94.95) (end 186.81 93.91) (width 0.2) (layer "F.Cu") (net 63))
-  (segment (start 186.81 93.91) (end 184.535 93.91) (width 0.2) (layer "F.Cu") (net 63))
   (segment (start 192.7075 92.838347) (end 192.622741 92.753588) (width 0.2) (layer "F.Cu") (net 63))
-  (segment (start 192.217013 94.95) (end 187.85 94.95) (width 0.2) (layer "F.Cu") (net 63))
   (segment (start 192.729511 92.12598) (end 192.7075 92.147991) (width 0.2) (layer "F.Cu") (net 63))
   (segment (start 192.622741 92.753588) (end 192.7075 92.668829) (width 0.2) (layer "F.Cu") (net 63))
+  (segment (start 184.535 93.91) (end 185.575 94.95) (width 0.2) (layer "F.Cu") (net 63))
   (segment (start 191.41 90.701562) (end 191.41 89.951) (width 0.2) (layer "F.Cu") (net 63))
   (segment (start 192.41 90.77) (end 192.729511 91.089511) (width 0.2) (layer "F.Cu") (net 63))
-  (segment (start 192.547013 94.62) (end 192.217013 94.95) (width 0.2) (layer "F.Cu") (net 63))
   (segment (start 193.257013 93.91) (end 199.78 93.91) (width 0.2) (layer "F.Cu") (net 63))
   (segment (start 191.185489 92.345264) (end 191.185489 90.926073) (width 0.2) (layer "F.Cu") (net 63))
@@
   (segment (start 192.7075 93.847991) (end 192.7075 92.838347) (width 0.2) (layer "F.Cu") (net 63))
   (segment (start 192.41 89.951) (end 192.41 90.77) (width 0.2) (layer "F.Cu") (net 63))
+  (segment (start 192.547013 94.62) (end 192.217013 94.95) (width 0.2) (layer "F.Cu") (net 63))
   (via (at 192.622741 92.753588) (size 0.6) (drill 0.3) (layers "F.Cu" "B.Cu") (net 63))
   (via (at 191.003929 92.526824) (size 0.6) (drill 0.3) (layers "F.Cu" "B.Cu") (net 63))
@@
   (segment (start 189.76 91.03) (end 187.06 91.03) (width 0.25) (layer "B.Cu") (net 65))
   (segment (start 194.57 91.03) (end 194.57 91.04) (width 0.25) (layer "B.Cu") (net 65))
-  (segment (start 187.41 92.7075) (end 187.4525 92.7075) (width 0.2) (layer "F.Cu") (net 66))
   (segment (start 189.94 93.05) (end 189.7 93.05) (width 0.2) (layer "F.Cu") (net 66))
+  (segment (start 185.87 91.57) (end 185.87 91.834933) (width 0.2) (layer "F.Cu") (net 66))
+  (segment (start 184.535 88.83) (end 185.87 90.165) (width 0.2) (layer "F.Cu") (net 66))
   (segment (start 194.94 93.05) (end 195.14 92.85) (width 0.2) (layer "F.Cu") (net 66))
   (segment (start 199.78 88.83) (end 199.78 89.800913) (width 0.2) (layer "F.Cu") (net 66))
   (segment (start 192.17 93.922991) (end 192.17 94.347013) (width 0.2) (layer "F.Cu") (net 66))
   (segment (start 189.7 93.05) (end 189.39 92.74) (width 0.2) (layer "F.Cu") (net 66))
-  (segment (start 184.535 88.83) (end 184.535 89.408875) (width 0.2) (layer "F.Cu") (net 66))
+  (segment (start 187.53 93.6675) (end 187.53 93.494933) (width 0.2) (layer "F.Cu") (net 66))
+  (segment (start 185.87 90.165) (end 185.87 91.57) (width 0.2) (layer "F.Cu") (net 66))
   (segment (start 192.027013 94.49) (end 191.42 94.49) (width 0.2) (layer "F.Cu") (net 66))
   (segment (start 195.41 89.951) (end 195.41 91.3845) (width 0.2) (layer "F.Cu") (net 66))
@@
   (segment (start 194.399916 93.05) (end 194.94 93.05) (width 0.2) (layer "F.Cu") (net 66))
   (segment (start 191.42 94.49) (end 190.52 94.49) (width 0.2) (layer "F.Cu") (net 66))
-  (segment (start 187.4525 92.7075) (end 188.09 92.07) (width 0.2) (layer "F.Cu") (net 66))
   (segment (start 190.52 94.49) (end 190.26 94.23) (width 0.2) (layer "F.Cu") (net 66))
-  (segment (start 187.196125 92.07) (end 188.09 92.07) (width 0.2) (layer "F.Cu") (net 66))
+  (segment (start 185.87 91.834933) (end 186.932422 92.897355) (width 0.2) (layer "F.Cu") (net 66))
+  (segment (start 187.53 93.494933) (end 186.932422 92.897355) (width 0.2) (layer "F.Cu") (net 66))
   (segment (start 196.730913 92.85) (end 195.14 92.85) (width 0.2) (layer "F.Cu") (net 66))
   (segment (start 199.78 89.800913) (end 196.730913 92.85) (width 0.2) (layer "F.Cu") (net 66))
   (segment (start 188.91 89.951) (end 188.91 91.44) (width 0.2) (layer "F.Cu") (net 66))
   (segment (start 192.17 94.347013) (end 192.027013 94.49) (width 0.2) (layer "F.Cu") (net 66))
-  (segment (start 184.535 89.408875) (end 187.196125 92.07) (width 0.2) (layer "F.Cu") (net 66))
   (segment (start 188.91 91.44) (end 188.7 91.65) (width 0.2) (layer "F.Cu") (net 66))
   (via (at 195.75 91.7245) (size 0.6) (drill 0.3) (layers "F.Cu" "B.Cu") (net 66))
+  (via (at 186.932422 92.897355) (size 0.6) (drill 0.3) (layers "F.Cu" "B.Cu") (net 66))
   (via (at 189.39 92.74) (size 0.6) (drill 0.3) (layers "F.Cu" "B.Cu") (net 66))
-  (via (at 188.09 92.07) (size 0.6) (drill 0.3) (layers "F.Cu" "B.Cu") (net 66))
   (via (at 195.14 92.85) (size 0.6) (drill 0.3) (layers "F.Cu" "B.Cu") (net 66))
   (via (at 190.26 94.23) (size 0.6) (drill 0.3) (layers "F.Cu" "B.Cu") (net 66))
@@
     (polygon
       (pts
-        (xy 175.12 72.61)
-        (xy 169.53 132.08)
-        (xy 122.26 136.14)
-        (xy 121.54 69.46)
+        (xy 115.320772 71.993074)
+        (xy 109.730772 131.463074)
+        (xy 62.460772 135.523074)
+        (xy 61.740772 68.843074)
+      )
+    )
+  )
+  (zone (net 2) (net_name "GND") (layer "F.Cu") (name "3V3") (hatch edge 0.508)
+    (connect_pads yes (clearance 0.15))
+    (min_thickness 0.15) (filled_areas_thickness no)
+    (fill yes (thermal_gap 0.15) (thermal_bridge_width 0.4))
+    (polygon
+      (pts
+        (xy 171.34 103.83)
+        (xy 155.55 103.42)
+        (xy 155.48 92.24)
+        (xy 173.28 86.46)
+      )
+    )
+  )
+  (zone (net 2) (net_name "GND") (layer "F.Cu") (name "3V3") (hatch edge 0.508)
+    (connect_pads yes (clearance 0.15))
+    (min_thickness 0.15) (filled_areas_thickness no)
+    (fill yes (thermal_gap 0.15) (thermal_bridge_width 0.4))
+    (polygon
+      (pts
+        (xy 166.900099 94.008326)
+        (xy 149.25 93.89)
+        (xy 149.22 100.2)
+        (xy 166.43 99.98)
+        (xy 168.41 123.87)
+        (xy 153.55 134.86)
+        (xy 117.6 122.17)
+        (xy 129.24 76.61)
+        (xy 172.7 75.39)
+      )
+    )
+  )
+  (zone (net 2) (net_name "GND") (layer "B.Cu") (name "3V3") (hatch edge 0.508)
+    (connect_pads yes (clearance 0.15))
+    (min_thickness 0.15) (filled_areas_thickness no)
+    (fill yes (thermal_gap 0.15) (thermal_bridge_width 0.4))
+    (polygon
+      (pts
+        (xy 174.27 130.96)
+        (xy 125.59 130.48)
+        (xy 125.59 130.42)
+        (xy 122.95 90.51)
+        (xy 128.39 75.38)
+        (xy 174.7 75.38)
       )
     )

Commit message: silkscreen
Parts:
- removed rb_cake: G*****, 0xB2_drawings:rb_cake
- removed splinky: G*****, 0xB2_drawings:splinky
- moved kibuzzard-6208EFFE 23.1 mm to (160.4, 94.4), turned to -90 degrees
- moved kibuzzard-61F01B61 22.6 mm to (160.4, 93.9), turned to 90 degrees
Other:
- board text added: "v1.0a"
- board text removed: "0xB2"
- board text removed: "bk3.1"

Commit message: silkscreen
Parts:
- removed SW1, SW3: SW_SPST, Library:PushSwitch
- added G***: LOGO, local-libraries:LOGO, B.Cu at (150.9, 97.5)
- added J13: Conn_01x02_Female, drawings:PinHeader_1x02_P1.27mm_Vertical, F.Cu at (157.9, 104.5)
- added kibuzzard-61F01940: G***, kibuzzard-61F01940, F.Cu at (149.1, 111.2)
- added kibuzzard-61F01940: G***, kibuzzard-61F01940, B.Cu at (149.0, 111.2)
- added kibuzzard-61F01957: G***, kibuzzard-61F01957, F.Cu at (140.0, 111.2)
- added kibuzzard-61F01957: G***, kibuzzard-61F01957, B.Cu at (140.0, 111.3)
- added kibuzzard-61F019CB: G***, kibuzzard-61F019CB, F.Cu at (142.1, 106.1)
- added kibuzzard-61F019CB: G***, kibuzzard-61F019CB, B.Cu at (142.2, 106.2)
- J1: footprint 0xLib_USB_Type-C:USB_C_Receptacle_HRO_TYPE-C-31-M-14 -> drawings:GT-USB-7014C
- J12, J2, J3, J4: footprint Connector_PinSocket_2.54mm:PinSocket_1x04_P2.54mm_Vertical -> drawings:PinHeader_1x04_P2.54mm_Vertical
- J5: footprint Connector_PinHeader_1.27mm:PinHeader_1x02_P1.27mm_Vertical -> drawings:PinHeader_1x02_P1.27mm_Vertical
- moved J1 6.95 mm to (192.2, 81.6)
Connections:
- net Rst renamed /~{RESET}
Routing:
- net /~{RESET}: track 48.9 -> 8.01 mm, vias 3 -> 1
- net /Gnd_daughter: track 20.7 -> 22.8 mm
- net /Vbus_daughter: track 25.0 -> 27.1 mm
- net /D-_daughter: track 27.2 -> 29.2 mm
- net /D+_daughter: track 25.6 -> 27.6 mm
- net Net-(J1-PadB5): track 2.27 -> 3.29 mm
- net Net-(J1-PadA5): track 2.65 -> 3.67 mm
Other:
- outline, holes or cut-outs redrawn
- board text added: "5V"
- board text added: "BASTARDKB.COM"
- board text added: "C1"
- board text added: "C2"
- board text added: "C3"
- board text added: "C4"
- board text added: "C5"
- board text added: "C6"
- board text added: "CS"
- board text added: "DIN"
- board text added: "GITHUB.COM/BASTARDKB"
- board text added: "GND"
- board text added: "MISO"
- board text added: "MOSI"
- board text added: "R1"
- board text added: "R2"
- board text added: "R3"
- board text added: "R4"
- board text added: "R5"
- board text added: "RST"
- board text added: "SCLK"

Commit message: silkscreen
Other:
- board text added: "SPLINKY-SHIELD"
Changed lines of the file:
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@@
     (effects (font (size 0.8 0.8) (thickness 0.15)) (justify mirror))
   )
-  (gr_text "BASTARDKB.COM" (at 135.84 97.68 90) (layer "B.SilkS")
+  (gr_text "BASTARDKB.COM" (at 135.96 96.76 90) (layer "B.SilkS")
     (effects (font (size 0.8 0.8) (thickness 0.12)) (justify mirror))
   )
@@
   (gr_text "CS" (at 142.298595 116.1 -45) (layer "B.SilkS")
     (effects (font (size 0.8 0.8) (thickness 0.15)) (justify mirror))
+  )
+  (gr_text "SPLINKY-SHIELD" (at 137.24 96.77 90) (layer "B.SilkS")
+    (effects (font (size 0.8 0.8) (thickness 0.12)) (justify mirror))
   )
   (gr_text "C3" (at 149.07 113.6 -45) (layer "B.SilkS")
@@
     (effects (font (size 0.6 0.6) (thickness 0.15)) (justify mirror))
   )
-  (gr_text "GITHUB.COM/BASTARDKB" (at 134.37 98 90) (layer "B.SilkS")
+  (gr_text "GITHUB.COM/BASTARDKB" (at 134.49 97.08 90) (layer "B.SilkS")
     (effects (font (size 0.8 0.8) (thickness 0.12)) (justify mirror))
   )
