File: splinktegrated.kicad_sch (KiCad schematic)
At the start: 65 parts, among them J1 USB_C_Receptacle_USB2.0, J10 NA_Ribbon, J11 NA_Serial, J12 NA_Conn_01x04_Female, J13 Conn_01x01_Socket, J14 Cirque, J15 Conn_01x01_Socket, J16 Conn_01x01_Socket, J17 Conn_01x01_Socket, J2 NA_Conn_01x04_Female, J3 NA_Conn_01x04_Female, J4 NA_Conn_01x04_Female, J5 Conn_01x02, J6 Cirque, J7 NA_trackball, J8 NA_Ribbon, J9 NA_RGB, SW1 NA_SW_SPST, SW2 NA_SW_SPST, U1 RP2040, U2 USBLC6-2P6, U3 XC6210B332MR-G, U4 USBLC6-2P6, U5 W25Q128JVS, Y1 Crystal_GND24

Commit message: schematic
Parts:
- removed FB1: FerriteBead_Small, Inductor_SMD:L_0603_1608Metric, symbol Device:FerriteBead_Small
- removed J1: USB_C_Receptacle_USB2.0, drawings:GT-USB-7014C, symbol Connector:USB_C_Receptacle_USB2.0
- removed J2, J3: NA_Conn_01x04_Female, Library:PinHeader_1x04_P2.54mm_Vertical_USB, symbol Connector:Conn_01x04_Female
- removed R4, R5: 5.1k, Resistor_SMD:R_0402_1005Metric, symbol Device:R
- removed U4: USBLC6-2P6, Package_TO_SOT_SMD:SOT-666, symbol Power_Protection:USBLC6-2P6
Connections:
- no-connect marks 12 -> 10
Other:
- note removed: "ESD protection"
- note removed: "Headers"
- note removed: "USB-C connector"

Commit message: move to usb c serial
Parts:
- removed J11: NA_Serial, drawings:Jack_3.5mm_PJ320E_Horizontal_custom, symbol Connector:AudioJack4
- removed J12, J4: NA_Conn_01x04_Female, drawings:PinHeader_1x04_P2.54mm_Vertical, symbol Connector:Conn_01x04_Female
- removed NA_J6: Serial, drawings:Jack_3.5mm_PJ320E_Horizontal_custom, symbol Connector:AudioJack4
- removed NA_JP1, NA_JP2: NA_Jumper_2_Open, local-libraries:SolderJumper-2_P1.3mm_Open_RoundedPad1.0x1.5mm, symbol Jumper:Jumper_2_Open
- removed NA_JP8, NA_JP9: NA_Jumper_2_Open, local-libraries:SolderJumper-2_P1.3mm_Open_TrianglePad1.0x1.5mm, symbol Jumper:Jumper_2_Open
- added FB1, FB2: FerriteBead_Small, Inductor_SMD:L_0603_1608Metric, symbol Device:FerriteBead_Small
- added J1, J18: USB_C_Receptacle_USB2.0, drawings:GT-USB-7014C, symbol Connector:USB_C_Receptacle_USB2.0
- added R4, R5: 5.1k, Resistor_SMD:R_0402_1005Metric, symbol Device:R
- added U4: USBLC6-2P6, Package_TO_SOT_SMD:SOT-666, symbol Power_Protection:USBLC6-2P6
Connections:
- net +3V3: now also J18.A4 (VBUS), J18.A9 (VBUS), J18.B4 (VBUS), J18.B9 (VBUS)
- net D+: now also J1.A6 (D+), J1.B6 (D+), U4.3 (I/O2), U4.4 (I/O2)
- net D-: now also J1.A7 (D-), J1.B7 (D-), U4.1 (I/O1), U4.6 (I/O1)
- net GND: now also FB1.1, FB2.1, J1.A1 (GND), J1.A12 (GND), J1.B1 (GND), J1.B12 (GND), J18.A1 (GND), J18.A12 (GND), J18.B1 (GND), J18.B12 (GND), R4.2, R5.2, U4.2 (GND)
- net VBUS: now also J1.A4 (VBUS), J1.A9 (VBUS), J1.B4 (VBUS), J1.B9 (VBUS), U4.5 (VBUS)
- net serial_l: now also J18.A6 (D+), J18.B6 (D+)
- net serial_l2: now also J18.A7 (D-), J18.B7 (D-)
- new net: J1.A5 (CC1), R4.1
- new net: FB2.2, J18.S1 (SHIELD)
- new net: J1.B5 (CC2), R5.1
- new net: FB1.2, J1.S1 (SHIELD)
- no-connect marks 10 -> 16
Other:
- note added: "ESD protection"
- note added: "Headers"
- note added: "Serial connector"
- note added: "USB-C connector"
- moved on the sheet: D2, F1, U2

Commit message: 5V interconnect
Parts:
- added D39: SMF5.0CA, reversible-kicad-footprints:D_SOD-123, symbol Device:D_TVS
- added F2: 1.5A 1206 Polyfuse, reversible-kicad-footprints:Fuse_1206_3216Metric, symbol Device:Polyfuse
- added FB13: 4A/0805, reversible-kicad-footprints:L-0805_2012Metric, symbol Device:Ferrite_Bead_Small
- added Q4: AO3401A, reversible-kicad-footprints:SOT-23-3, symbol Transistor_FET:AO3401A
Connections:
- net +3V3: no longer J18.A4 (VBUS), J18.A9 (VBUS), J18.B4 (VBUS), J18.B9 (VBUS)
- net +5V: now also Q4.2 (S)
- net GND: now also D39.2 (A2), Q4.1 (G)
- new net: D39.1 (A1), F2.1, Q4.3 (D)
- new net: F2.2, FB13.2
- new net: FB13.1, J18.A4 (VBUS), J18.A9 (VBUS), J18.B4 (VBUS), J18.B9 (VBUS)
Other:
- note added: "Old"
- note removed: "Headers"
- moved on the sheet: U4

Commit message: oops
Connections:
- net VBUS: now also FB13.1, J18.A4 (VBUS), J18.A9 (VBUS), J18.B4 (VBUS), J18.B9 (VBUS)
Changed lines of the file:
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@@
 	)
 	(junction
+		(at -152.4 26.67)
+		(diameter 0)
+		(color 0 0 0 0)
+	)
+	(junction
 		(at 33.02 115.57)
 		(diameter 0)
@@
 	(wire
 		(pts
+			(xy -152.4 26.67) (xy -151.13 26.67)
+		)
+		(stroke
+			(width 0)
+			(type default)
+		)
+	)
+	(wire
+		(pts
 			(xy 228.6 64.77) (xy 237.49 64.77)
 		)
@@
 	(wire
 		(pts
+			(xy -152.4 21.59) (xy -152.4 26.67)
+		)
+		(stroke
+			(width 0)
+			(type default)
+		)
+	)
+	(wire
+		(pts
 			(xy 182.88 73.66) (xy 191.77 73.66)
 		)
@@
 	(wire
 		(pts
-			(xy -153.67 26.67) (xy -151.13 26.67)
+			(xy -153.67 26.67) (xy -152.4 26.67)
 		)
 		(stroke
@@
 					(unit 1)
 				)
+			)
+		)
+	)
+	(symbol
+		(lib_id "power:VBUS")
+		(at -152.4 21.59 0)
+		(unit 1)
+		(exclude_from_sim no)
+		(in_bom yes)
+		(on_board yes)
+		(dnp no)
+		(property "Reference" "#PWR0105"
+			(at -152.4 25.4 0)
+			(effects
+				(font
+					(size 1.27 1.27)
+				)
+				(hide yes)
+			)
+		)
+		(property "Value" "VBUS"
+			(at -152.4 17.78 0)
+			(effects
+				(font
+					(size 1.27 1.27)
+				)
+			)
+		)
+		(property "Footprint" ""
+			(at -152.4 21.59 0)
+			(effects
+				(font
+					(size 1.27 1.27)
+				)
+				(hide yes)
+			)
+		)
+		(property "Datasheet" ""
+			(at -152.4 21.59 0)
+			(effects
+				(font
+					(size 1.27 1.27)
+				)
+				(hide yes)
+			)
+		)
+		(property "Description" ""
+			(at -152.4 21.59 0)
+			(effects
+				(font
+					(size 1.27 1.27)
+				)
+				(hide yes)
+			)
+		)
+		(pin "1"
+		)
+		(instances
+			(project "splinktegrated"
+				(path "/7353e96a-343a-4876-b497-b1d205a14d97"
+					(reference "#PWR0105")
+					(unit 1)
+				)

Commit message: move components around
Parts:
- removed D39: SMF5.0CA, reversible-kicad-footprints:D_SOD-123, symbol Device:D_TVS
- added D3: B5817, Diode_SMD:D_SOD-323, symbol Device:D_Schottky
- added Q5: AO3401A, reversible-kicad-footprints:SOT-23-3, symbol Transistor_FET:AO3401A
Connections:
- net GND: now also Q5.1 (G)
- net VBUS: now also C1.1, D2.1 (K), NA_JP5.1 (A), U3.1 (VIN), U3.3 (EN), D3.1 (K); no longer F1.1, FB13.1, J1.A4 (VBUS), J1.A9 (VBUS), J1.B4 (VBUS), J1.B9 (VBUS), J18.A4 (VBUS), J18.A9 (VBUS), J18.B4 (VBUS), J18.B9 (VBUS), R10.2
- net at F1.2: now also Q5.3 (D); no longer D2.2 (A)
- removed net +5V: C1.1, D2.1 (K), NA_JP5.1 (A), Q4.2 (S), U3.1 (VIN), U3.3 (EN)
- new net: FB13.1, J18.A4 (VBUS), J18.A9 (VBUS), J18.B4 (VBUS), J18.B9 (VBUS)
- new net: F1.1, J1.A4 (VBUS), J1.A9 (VBUS), J1.B4 (VBUS), J1.B9 (VBUS)
- new net: D3.2 (A), Q4.2 (S)
- new net V_USB_DETECT: D2.2 (A), Q5.2 (S), R10.2
Other:
- moved on the sheet: F1, Q4

Commit message: BOM work
Parts:
- F2: value 1.5A 1206 Polyfuse -> Polyfuse; footprint reversible-kicad-footprints:Fuse_1206_3216Metric -> Fuse:Fuse_0603_1608Metric; LCSC (none) -> C69679
Changed lines of the file:
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@@
 			)
 		)
-		(property "Value" "1.5A 1206 Polyfuse"
+		(property "Value" "Polyfuse"
 			(at -140.97 30.0736 90)
 			(effects
@@
 			)
 		)
-		(property "Footprint" "reversible-kicad-footprints:Fuse_1206_3216Metric"
+		(property "Footprint" "Fuse:Fuse_0603_1608Metric"
 			(at -146.05 25.4 0)
 			(effects
@@
 			(at -140.97 26.67 0)
 			(effects
+				(font
+					(size 1.27 1.27)
+				)
+			)
+		)
+		(property "LCSC" "C69679"
+			(at -140.97 26.67 0)
+			(effects

Commit message: placement and routing
Parts:
- D2, D3: footprint Diode_SMD:D_SOD-323 -> local-libraries:D_SOD-323
- FB13: footprint reversible-kicad-footprints:L-0805_2012Metric -> Inductor_SMD:L_0603_1608Metric; LCSC (none) -> C98288
- Q4, Q5: footprint reversible-kicad-footprints:SOT-23-3 -> local-libraries:TSOT-23; LCSC (none) -> AO3401A
- U4: LCSC (none) -> C2827693
Connections:
- net +3V3: no longer J9.1 (Pin_1)
- net VBUS: now also J9.1 (Pin_1)
Other:
- note removed: "Serial and protection"
Changed lines of the file:
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@@
 		)
 	)
-	(rectangle
-		(start 298.45 82.55)
-		(end 392.43 234.95)
-		(stroke
-			(width 0)
-			(type default)
-		)
-		(fill
-			(type none)
-		)
-	)
 	(text "Hand"
 		(exclude_from_sim no)
@@
 		)
 	)
-	(text "Serial and protection"
-		(exclude_from_sim no)
-		(at 298.45 81.28 0)
-		(effects
-			(font
-				(size 1.778 1.778)
-				(thickness 0.3556)
-				(bold yes)
-			)
-			(justify left bottom)
-		)
-	)
 	(text "Indicator & buttons"
 		(exclude_from_sim no)
@@
 			)
 		)
-		(property "Footprint" "reversible-kicad-footprints:L-0805_2012Metric"
+		(property "Footprint" "Inductor_SMD:L_0603_1608Metric"
 			(at -148.59 28.448 90)
 			(effects
@@
 			)
 		)
+		(property "LCSC" "C98288"
+			(at -148.59 26.67 0)
+			(effects
+				(font
+					(size 1.27 1.27)
+				)
+			)
+		)
 		(pin "1"
 		)
@@
 			)
 		)
-		(property "Footprint" "reversible-kicad-footprints:SOT-23-3"
+		(property "Footprint" "local-libraries:TSOT-23"
 			(at -45.72 27.94 0)
 			(effects
@@
 			)
 		)
+		(property "LCSC" "AO3401A"
+			(at -43.18 22.86 0)
+			(effects
+				(font
+					(size 1.27 1.27)
+				)
+			)
+		)
 		(pin "1"
 		)
@@
 			)
 		)
-		(property "Footprint" "Diode_SMD:D_SOD-323"
+		(property "Footprint" "local-libraries:D_SOD-323"
 			(at -121.92 26.67 0)
 			(effects
@@
 			)
 		)
-		(property "Value" "+3V3"
+		(property "Value" "VBUS"
 			(at 330.2 26.67 0)
 			(effects
@@
 			)
 		)
-		(property "Footprint" "reversible-kicad-footprints:SOT-23-3"
+		(property "Footprint" "local-libraries:TSOT-23"
 			(at -134.62 29.21 0)
 			(effects
@@
 			)
 		)
+		(property "LCSC" "AO3401A"
+			(at -132.08 24.13 0)
+			(effects
+				(font
+					(size 1.27 1.27)
+				)
+			)
+		)
 		(pin "1"
 		)
@@
 			)
 		)
+		(property "LCSC" "C2827693"
+			(at -66.04 99.06 0)
+			(effects
+				(font
+					(size 1.27 1.27)
+				)
+			)
+		)
 		(pin "1"
 		)
@@
 			)
 		)
-		(property "Footprint" "Diode_SMD:D_SOD-323"
+		(property "Footprint" "local-libraries:D_SOD-323"
 			(at -31.75 25.4 0)
 			(effects

Commit message: add serial breakout
Parts:
- added FB14: 4A/0805, Inductor_SMD:L_0603_1608Metric, symbol Device:Ferrite_Bead_Small
- added J19, J20: Conn_01x01_Socket, local-libraries:PinHeader_1x01_P1.27mm_Vertical, symbol Connector:Conn_01x01_Socket
Connections:
- net serial_l: now also J19.1 (Pin_1)
- net serial_l2: now also J20.1 (Pin_1)
- net at J1.A4 (VBUS), J1.A9 (VBUS), J1.B4 (VBUS)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: now also FB14.1; no longer F1.1
- new net: F1.1, FB14.2
Other:
- moved on the sheet: D2, F1, J13, J15, J16, J17, NA_JP6, NA_JP7, Q5, R12
