File: right/splinktegrated.kicad_sch (KiCad schematic)
At the start: 66 parts, among them J1 USB_C_Receptacle_USB2.0, J10 NA_Ribbon, J13 Conn_01x01_Socket, J14 Cirque, J15 Conn_01x01_Socket, J16 Conn_01x01_Socket, J17 Conn_01x01_Socket, J18 USB_C_Receptacle_USB2.0, J19 Conn_01x01_Socket, J20 Conn_01x01_Socket, J5 Conn_01x02, J6 Cirque, J7 NA_trackball, J8 NA_Ribbon, J9 NA_RGB, Q4 AO3401A, Q5 AO3401A, SW1 NA_SW_SPST, SW2 NA_SW_SPST, U1 RP2040, U2 USBLC6-2P6, U3 XC6210B332MR-G, U4 USBLC6-2P6, U5 W25Q128JVS, U6 74LVC1T45, Y1 Crystal_GND24

Commit message: start renaming right side labels for later incorporation
Parts:
- renumbered NA_JP6 to NA_JP1, SW2 to SW9001, SW1 to SW9002, C1 to right_C9000, C8 to right_C9001, C9 to right_C9002, C11 to right_C9003, C12 to right_C9004, C13 to right_C9005, C14 to right_C9006, C10 to right_C9007, C2 to right_C9008, C3 to right_C9009, C4 to right_C9010, C5 to right_C9011, C6 to right_C9012, C7 to right_C9013, D39 to right_D9000, D2 to right_D9001, D1 to right_D9002, F2 to right_F9000, F1 to right_F9001, FB13 to right_FB9000, FB1 to right_FB9001, FB2 to right_FB9002, FB14 to right_FB9003, H2 to right_H9001, H1 to right_H9003, J18 to right_J9000, J1 to right_J9001, J20 to right_J9002, J19 to right_J9003, J5 to right_J9004, J8 to right_J9005, J9 to right_J9006, J10 to right_J9007, J7 to right_J9008, J15 to right_J9009, J14 to right_J9010, J17 to right_J9011, J16 to right_J9012, J13 to right_J9013, J6 to right_J9014, NA_JP5 to right_NA_JP9000, NA_JP7 to right_NA_JP9001, Q5 to right_Q9000, Q4 to right_Q9001, R5 to right_R9000, R4 to right_R9001, R1 to right_R9002, R2 to right_R9003, R3 to right_R9004, R6 to right_R9005, R7 to right_R9006, R8 to right_R9007, R9 to right_R9008, R10 to right_R9009, R11 to right_R9010, R12 to right_R9011, U3 to right_U9000, U6 to right_U9001, U2 to right_U9002, U4 to right_U9003, U5 to right_U9004, U1 to right_U9005, Y1 to right_Y9000

Commit message: start renaming nets
Connections:
- net +3V3 renamed right_+3V3
- net D+ renamed D+_daughter
- net D- renamed D-_daughter
- net GND renamed right_GND
- net QSPI_D0 renamed right_QSPI_D0
- net QSPI_D1 renamed right_QSPI_D1
- net QSPI_D2 renamed right_QSPI_D2
- net QSPI_D3 renamed right_QSPI_D3
- net QSPI_SCLK renamed right_QSPI_SCLK
- net QSPI_~{CS} renamed right_QSPI_~{CS}
- net VBUS renamed right_VBUS
- net V_USB_DETECT renamed right_V_USB_DETECT
- net serial_l renamed right_serial_l
- net serial_l2 renamed right_serial_l2
- net ~{RESET} renamed right_~{RESET}
Other:
- note added: "- Transistor for protection against shorts between power and right_GND (reverse polarity) - TVS diode against power surges - U2 for ESD protection On the serial port, we use a TVS diode instead of Zener (on the main connector) to avoid power drop, as power would have to go through 2 Zener - one reversed."
- note added: "The datasheet of the SK6815 Mini-E mentions that: - Vdd > 3.7V, hence we use the right_VBUS here which is around 4.7V - Vih >= 0.7*Vdd = 0.7*4.7 = 3.29V Technically here Vih is at 3.3V as it's output by the RP2040. But as a precaution, we shift it to the right_VBUS levels. Vin: logic input voltage Vdd: power supply Vih: input signal flip treshold"
- note removed: "- Transistor for protection against shorts between power and Gnd (reverse polarity) - TVS diode against power surges - U2 for ESD protection On the serial port, we use a TVS diode instead of Zener (on the main connector) to avoid power drop, as power would have to go through 2 Zener - one reversed."
- note removed: "The datasheet of the SK6815 Mini-E mentions that: - Vdd > 3.7V, hence we use the Vbus here which is around 4.7V - Vih >= 0.7*Vdd = 0.7*4.7 = 3.29V Technically here Vih is at 3.3V as it's output by the RP2040. But as a precaution, we shift it to the VBus levels. Vin: logic input voltage Vdd: power supply Vih: input signal flip treshold"

Commit message: nets
Connections:
- net D10 renamed right_D10
- net D11 renamed right_D11
- net D13 renamed right_D13
- net D14 renamed right_D14
- net LED renamed right_LED
- net SCL renamed right_SCL
- net SDA renamed right_SDA
- net VBUS_DET renamed right_VBUS_DET
- net col1_l renamed right_col1_l
- net col2_l renamed right_col2_l
- net col3_l renamed right_col3_l
- net col4_l renamed right_col4_l
- net col5_l renamed right_right_col5_l
- net col6_l renamed right_col6_l
- net hand renamed right_hand
- net miso_l renamed right_MISO_l
- net mosi_l renamed right_MOSI_l
- net rgb_3v3 renamed right_rgb_3v3
- net right_QSPI_SCLK renamed right_QSPI_right_SCLK
- net row1_l renamed right_row1_l
- net row2_l renamed right_row2_l
- net row3_l renamed right_row3_l
- net row4_l renamed right_row4_l
- net row5_l renamed right_row5_l
- net sc_l renamed right_sc_l
- net ss_l renamed right_ss_l
Other:
- note added: "right_LED signal"
- note added: "right_hand"
- note removed: "Hand"
- note removed: "LED signal"
